File: hardware/L4.kicad_sch (KiCad schematic)
At the start: 124 parts, among them J1 JST_PH, J2 JST_PH, Q1 SSM3J332R, Q2 SSM3J332R, SW1 SW_Push, SW10 SW_Push, SW11 SW_Push, SW12 SW_Push, SW13 SW_Push, SW14 SW_Push, SW15 SW_Push, SW16 SW_Push, SW17 SW_Push, SW18 SW_Push, SW19 SW_Push, SW2 SW_Push, SW20 SW_Push, SW21 SW_Push, SW22 SW_Push, SW23 SW_Push, SW24 SW_Push, SW25 SW_Push, SW26 SW_Push, SW27 SW_DP3T, SW28 SW_Push, SW29 SW_Push, SW3 SW_Push, SW30 SW_Push, SW31 SW_Push, SW32 SW_Push, SW33 SW_Push, SW34 SW_Push, SW35 SW_Push, SW36 SW_Push, SW37 SW_Push, SW38 SW_Push, SW39 SW_Push, SW4 SW_Push, SW40 SW_Push, SW41 SW_Push, SW42 SW_Push, SW43 SW_Push, SW44 SW_Push, SW45 SW_Push, SW46 SW_Push, SW47 SW_Push, SW48 SW_Push, SW49 SW_Push, SW5 SW_Push, SW50 SW_Push, SW51 SW_Push, SW52 SW_Push, SW53 SW_Push, SW54 SW_DP3T, SW6 SW_Push, SW7 SW_Push, SW8 SW_Push, SW9 SW_Push, U1 XIAO nRF52840, U2 XIAO nRF52840

Commit message: finish part layout
Parts:
- removed R1, R2: 10k, Resistor_THT:R_Axial_DIN0207_L6.3mm_D2.5mm_P7.62mm_Horizontal, symbol Device:R
- SW27, SW54: footprint akizuki:MSS23D18 -> akizuki:SK23D07
Changed lines of the file:
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@@
   (junction (at 55.88 137.16) (diameter 0) (color 0 0 0 0)
   )
-  (junction (at 92.71 40.64) (diameter 0) (color 0 0 0 0)
-  )
   (junction (at 293.37 154.94) (diameter 0) (color 0 0 0 0)
   )
@@
   )
   (junction (at 66.04 144.78) (diameter 0) (color 0 0 0 0)
-  )
-  (junction (at 254 40.64) (diameter 0) (color 0 0 0 0)
   )
   (junction (at 111.76 162.56) (diameter 0) (color 0 0 0 0)
@@
     (stroke (width 0) (type default))
   )
-  (wire (pts (xy 92.71 41.91) (xy 92.71 40.64))
-    (stroke (width 0) (type default))
-  )
   (wire (pts (xy 116.84 119.38) (xy 116.84 137.16))
     (stroke (width 0) (type default))
@@
     (stroke (width 0) (type default))
   )
-  (wire (pts (xy 254 40.64) (xy 254 41.91))
-    (stroke (width 0) (type default))
-  )
   (wire (pts (xy 96.52 144.78) (xy 111.76 144.78))
     (stroke (width 0) (type default))
@@
     )
   )
-  (global_label "GND_R" (shape input) (at 254 49.53 270) (fields_autoplaced)
-    (effects (font (size 1.27 1.27)) (justify right))
-    (property "Intersheetrefs" "${INTERSHEET_REFS}" (at 254 58.6233 90)
-      (effects (font (size 1.27 1.27)) (justify right) hide)
-    )
-  )
   (global_label "VBUS_L" (shape input) (at 83.82 40.64 180) (fields_autoplaced)
     (effects (font (size 1.27 1.27)) (justify right))
@@
     (property "Intersheetrefs" "${INTERSHEET_REFS}" (at 224.6909 41.91 0)
       (effects (font (size 1.27 1.27)) (justify left) hide)
-    )
-  )
-  (global_label "GND_L" (shape input) (at 92.71 49.53 270) (fields_autoplaced)
-    (effects (font (size 1.27 1.27)) (justify right))
-    (property "Intersheetrefs" "${INTERSHEET_REFS}" (at 92.71 58.3814 90)
-      (effects (font (size 1.27 1.27)) (justify right) hide)
     )
   )
@@
       (effects (font (size 1.27 1.27)))
     )
-    (property "Footprint" "akizuki:MSS23D18" (at 89.535 28.575 0)
+    (property "Footprint" "akizuki:SK23D07" (at 89.535 28.575 0)
       (effects (font (size 1.27 1.27)) hide)
     )
@@
       (effects (font (size 1.27 1.27)))
     )
-    (property "Footprint" "akizuki:MSS23D18" (at 250.825 28.575 0)
+    (property "Footprint" "akizuki:SK23D07" (at 250.825 28.575 0)
       (effects (font (size 1.27 1.27)) hide)
     )
@@
     )
   )
-  (symbol (lib_id "Device:R") (at 92.71 45.72 0) (unit 1)
-    (in_bom yes) (on_board yes) (dnp no)
-    (property "Reference" "R1" (at 95.25 44.45 0)
-      (effects (font (size 1.27 1.27)) (justify left))
-    )
-    (property "Value" "10k" (at 95.25 46.99 0)
-      (effects (font (size 1.27 1.27)) (justify left))
-    )
-    (property "Footprint" "Resistor_THT:R_Axial_DIN0207_L6.3mm_D2.5mm_P7.62mm_Horizontal" (at 90.932 45.72 90)
-      (effects (font (size 1.27 1.27)) hide)
-    )
-    (property "Datasheet" "~" (at 92.71 45.72 0)
-      (effects (font (size 1.27 1.27)) hide)
-    )
-    (pin "1")
-    (pin "2")
-    (instances
-      (project "L4"
-        (path "/529e0543-76b7-4235-890e-1315675f8617"
-          (reference "R1") (unit 1)
-        )
-      )
-    )
-  )
   (symbol (lib_id "power:PWR_FLAG") (at 139.7 34.29 0) (unit 1)
     (in_bom yes) (on_board yes) (dnp no) (fields_autoplaced)
@@
       (effects (font (size 1.27 1.27)))
     )
-    (property "Footprint" "akizuki:MSS23D18" (at 130.175 29.845 0)
+    (property "Footprint" "akizuki:SK23D07" (at 130.175 29.845 0)
       (effects (font (size 1.27 1.27)) hide)
     )
@@
       (effects (font (size 1.27 1.27)))
     )
-    (property "Footprint" "akizuki:MSS23D18" (at 294.005 29.845 0)
+    (property "Footprint" "akizuki:SK23D07" (at 294.005 29.845 0)
       (effects (font (size 1.27 1.27)) hide)
     )
@@
         )
       )
-    )
-  )
-  (symbol (lib_id "Device:R") (at 254 45.72 0) (unit 1)
-    (in_bom yes) (on_board yes) (dnp no) (fields_autoplaced)
-    (property "Reference" "R2" (at 256.54 44.45 0)
-      (effects (font (size 1.27 1.27)) (justify left))
-    )
-    (property "Value" "10k" (at 256.54 46.99 0)
-      (effects (font (size 1.27 1.27)) (justify left))
-    )
-    (property "Footprint" "Resistor_THT:R_Axial_DIN0207_L6.3mm_D2.5mm_P7.62mm_Horizontal" (at 252.222 45.72 90)
-      (effects (font (size 1.27 1.27)) hide)
-    )
-    (property "Datasheet" "~" (at 254 45.72 0)
-      (effects (font (size 1.27 1.27)) hide)
-    )
-    (pin "1")
-    (pin "2")
-    (instances
-      (project "L4"
-        (path "/529e0543-76b7-4235-890e-1315675f8617"
-          (reference "R2") (unit 1)
-        )
-      )

Commit message: finish routing
Parts:
- C1, C2: value 4.7u -> 100u; footprint Capacitor_SMD:C_0805_2012Metric_Pad1.18x1.45mm_HandSolder -> Capacitor_SMD:C_1206_3216Metric_Pad1.33x1.80mm_HandSolder
Connections:
- net COL0_R: now also U2.7 (D6/1.11); no longer U2.6 (D5/0.05)
- net COL1_R: now also U2.6 (D5/0.05); no longer U2.7 (D6/1.11)
- net COL2_L: now also U1.11 (D10/1.15); no longer U1.8 (D7/1.12)
- net COL2_R: now also U2.5 (D4/0.04); no longer U2.8 (D7/1.12)
- net COL3_L: now also U1.10 (D9/1.14); no longer U1.9 (D8/1.13)
- net COL3_R: now also U2.8 (D7/1.12); no longer U2.9 (D8/1.13)
- net COL4_L: now also U1.9 (D8/1.13); no longer U1.10 (D9/1.14)
- net COL4_R: now also U2.9 (D8/1.13); no longer U2.10 (D9/1.14)
- net COL5_L: now also U1.8 (D7/1.12); no longer U1.11 (D10/1.15)
- net COL5_R: now also U2.10 (D9/1.14); no longer U2.11 (D10/1.15)
- net ROW0_R: now also U2.11 (D10/1.15); no longer U2.1 (D0/0.02)
- net ROW1_R: now also U2.1 (D0/0.02); no longer U2.2 (D1/0.03)
- net ROW2_R: now also U2.2 (D1/0.03); no longer U2.3 (D2/0.28)
- net ROW3_R: now also U2.3 (D2/0.28); no longer U2.4 (D3/0.29)
- net ROW4_R: now also U2.4 (D3/0.29); no longer U2.5 (D4/0.04)
